Commit message: Fix camera pose

File: urdf/setup.urdf.xacro (robot description, xacro)
@@ -7,10 +7,4 @@
     <xacro:property name="clip_near" value="0.1"/>
     <xacro:property name="clip_far" value="100"/>
-    <link name="world"/>
-    <joint name="box_mount" type="fixed">
-        <origin xyz="0 0 0.25"/>
-        <parent link="world"/>
-        <child link="box"/>
-    </joint>
     <link name="box">
         <inertial>
@@ -33,5 +27,5 @@
     <!-- Camera -->
     <joint name="fisheye_mount" type="fixed">
-        <origin xyz="0.05 0 0.2" rpy="0 0 ${pi}"/>
+        <origin xyz="0.05 0 0.2" rpy="0 0 0"/>
         <parent link="box"/>
         <child link="fisheye_camera"/>
@@ -39,4 +33,5 @@
     <link name="fisheye_camera">
         <visual>
+            <origin rpy="0 0 ${pi}"/>
             <geometry>
                 <mesh filename="package://ocam-calibration/meshes/camera.dae" scale="0.7 0.7 0.7"/>
@@ -90,28 +85,4 @@
         </sensor>
     </gazebo>
-    <!-- Chessboard -->
-    <joint name="chessboard_mount" type="fixed">
-        <origin xyz="1 0 0"/>
-        <parent link="box"/>
-        <child link="chessboard"/>
-    </joint>
-    <link name="chessboard">
-        <inertial>
-            <mass value="0.001"/>
-            <inertia ixx="1.0" ixy="0.0" ixz="0.0"
-                     iyy="1.0" iyz="0.0"
-                     izz="1.0"/>
-        </inertial>
-        <visual>
-            <geometry>
-                <box size="0.1 0.1 0.5"/>
-            </geometry>
-        </visual>
-        <collision>
-            <geometry>
-                <box size="0.1 0.1 0.5"/>
-            </geometry>
-        </collision>
-    </link>
     <gazebo>
         <static>true</static>

Commit message: Fix camera params

File: urdf/setup.urdf.xacro (robot description, xacro)
@@ -3,7 +3,8 @@
     <!-- camera props -->
     <xacro:property name="hfov" value="${radians(185)}"/>
-    <xacro:property name="width" value="${754}"/>
-    <xacro:property name="height" value="${480}"/>
-    <xacro:property name="clip_near" value="0.1"/>
+    <xacro:property name="fps" value="25"/>
+    <xacro:property name="width" value="754"/>
+    <xacro:property name="height" value="480"/>
+    <xacro:property name="clip_near" value="0.02"/>
     <xacro:property name="clip_far" value="100"/>
     <link name="box">
@@ -52,5 +53,5 @@
     <gazebo reference="fisheye_camera">
         <sensor name="fisheye" type="wideanglecamera">
-            <update_rate>25</update_rate>
+            <update_rate>${fps}</update_rate>
             <always_on>true</always_on>
             <camera>
@@ -72,5 +73,5 @@
                     <!--<cutoff_angle>${pi/2]</cutoff_angle>-->
                     <!-- resolution of the cube-map texture, the higher it is - the sharper is your image -->
-                    <env_texture_size>4096</env_texture_size>
+                    <env_texture_size>1024</env_texture_size>
                 </lens>
             </camera>
