Commit message: Fix

File: urdf/chessboard.urdf.xacro (robot description, xacro)
@@ -1,4 +1,11 @@
 <?xml version="1.0"?>
 <robot name="chessboard">
+    <!-- virtual link -->
+    <link name="world"/>
+    <joint name="chessboard_mount" type="fixed">
+        <origin xyz="0.3 0 0.45"/>
+        <parent link="world"/>
+        <child link="chessboard"/>
+    </joint>
     <link name="chessboard">
         <inertial>

File: urdf/setup.urdf.xacro (robot description, xacro)
@@ -65,13 +65,15 @@
                     <far>${clip_far}</far>
                 </clip>
+                <!-- See https://en.wikipedia.org/wiki/Fisheye_lens#Mapping_function -->
                 <lens>
+                    <!-- gnomonical, stereographic, equidistant, equisolid_angle, orthographic -->
                     <type>orthographic</type>
                     <!-- if it is set to `true` your horizontal FOV will remain as defined -->
                     <!-- otherwise it depends on lens type and custom function, if there is one -->
-                    <scale_to_hfov>false</scale_to_hfov>
+                    <scale_to_hfov>true</scale_to_hfov>
                     <!-- clip everything that is outside of this angle -->
-                    <!--<cutoff_angle>${pi/2]</cutoff_angle>-->
+                    <cutoff_angle>${pi/2]</cutoff_angle>
                     <!-- resolution of the cube-map texture, the higher it is - the sharper is your image -->
-                    <env_texture_size>1024</env_texture_size>
+                    <env_texture_size>512</env_texture_size>
                 </lens>
             </camera>
